File: ADC_fifo_buffer_eval_board/ADC_fifo_buffer_eval_board.kicad_sch (KiCad schematic)
At the start: 1 part, among them IC1 SN74V245-7PAG

Commit message: w
Parts:
- added C1: 22p_low_tolerance, symbol Device:C_Small
- added C10, C12, C14, C2, C3, C6, C8: 100n, symbol Device:C_Small
- added C11, C13, C15, C4, C5, C7, C9: 1u, symbol Device:C_Small
- added IC2: 74AHC1G86GV,125, SOT95P275X110-5N, symbol 74AHC1G86GV_125:74AHC1G86GV,125
- added IC3: MAX9010EXT+, SOT65P210X110-6N, symbol MAX9010EXT+:MAX9010EXT+
- added R1: 1.5k_low_tolerance, symbol Device:R_Small
- added R2, R3: 5.1k, symbol Device:R_Small
- added S1, S2, S3, S4, S5: ~, Trace_Shunt:Untitled, symbol Trace_Shunt:_1
Connections:
- net FIFO_D14_extra_write: now also IC1.2 (D14)
- net GND: now also C1.2, C10.2, C11.2, C12.2, C13.2, C14.2, C15.2, C2.1, C3.1, C4.1, C5.1, C6.2, C7.2, C8.2, C9.2, IC2.3 (GND), IC3.2 (GND), R3.2
- net VCC: now also R2.1; no longer IC1.22 (VCC_1), IC1.33 (VCC_2), IC1.43 (VCC_3), IC1.49 (VCC_4), IC1.56 (VCC_5), IC1.59 (~{LD})
- net Write_CLK: now also IC2.4 (Y)
- net FIFO_D12_extra_write renamed ADC_CLK
- net ADC_CLK: now also IC2.1 (B), R1.2
- new net: IC3.3 (IN+), R2.2, R3.1
- new net: IC2.2 (A), IC3.1 (OUT)
- new net: C1.1, IC3.4 (IN-), R1.1
- new net +3.3V: C2.2, C5.2, IC1.59 (~{LD}), IC3.5 (VCC_1), IC3.6 (VCC_2)
- new net +3.3v: C3.2, C4.2, IC2.5 (VCC), S1.1, S2.1, S3.1, S4.1, S5.1
- new net VCC1: C6.1, C7.1, IC1.22 (VCC_1), S5.2
- new net VCC2: C8.1, C9.1, IC1.33 (VCC_2), S4.2
- new net VCC3: C10.1, C11.1, IC1.43 (VCC_3), S3.2
- new net VCC4: C12.1, C13.1, IC1.49 (VCC_4), S2.2
- new net VCC5: C14.1, C15.1, IC1.56 (VCC_5), S1.2
Other:
- note added: "Should multiply to 20.0202020 MHz, as per equation R1*C1=(2/3)*(1/f_double)"

Commit message: w
Parts:
- added J1: 2-826942-0, 2-826942-0:HDRV40W63P254_2X20_5080X500X860P, symbol 2-826942-0:2-826942-0
Connections:
- net ADC_CLK: now also J1.6
- net ADC_DA0: now also J1.38
- net ADC_DA1: now also J1.36
- net ADC_DA10: now also J1.18
- net ADC_DA11: now also J1.16
- net ADC_DA2: now also J1.34
- net ADC_DA3: now also J1.32
- net ADC_DA4: now also J1.30
- net ADC_DA5: now also J1.28
- net ADC_DA6: now also J1.26
- net ADC_DA7: now also J1.24
- net ADC_DA8: now also J1.22
- net ADC_DA9: now also J1.20
- net GND: now also J1.10, J1.11, J1.13, J1.15, J1.17, J1.19, J1.21, J1.23, J1.25, J1.27, J1.29, J1.3, J1.31, J1.33, J1.35, J1.37, J1.39, J1.5, J1.7, J1.8, J1.9
- removed net FIFO_Q12_extra_read: IC1.45 (Q12), IC1.47 (Q13), IC1.48 (Q14), IC1.50 (Q15), IC1.52 (Q16), IC1.53 (Q17)
- new net DSP_Q12: IC1.45 (Q12)
- new net FIFO_Q13_extra_read: IC1.47 (Q13)
- new net FIFO_Q14_extra_read: IC1.48 (Q14)
- new net FIFO_Q15_extra_read: IC1.50 (Q15)
- new net FIFO_Q16_extra_read: IC1.52 (Q16)
- new net FIFO_Q17_extra_read: IC1.53 (Q17)
- new net OUTPUT_ENABLE: J1.40
- no-connect marks 3 -> 8
Other:
- note added: "ADC input header"
- note added: "Should multiply to 20.0202020 MHz, as per equation R1*C1=(2/3)*(1/f_double) design from: https://www.analog.com/en/resources/design-notes/simple-circuit-doubles-input-frequency.html"
- note added: "The 60 pin BTB connector is less readily available. We would need a mini PCB that is just the BTB connectior that routes the traces to other connectors mezzaniene that goes into a morecommon flat ribbon cable. and then go to another mezzanine on the FIFO PCB"
- note removed: "Should multiply to 20.0202020 MHz, as per equation R1*C1=(2/3)*(1/f_double)"
- moved on the sheet: C1, C2, C3, C4, C5, IC2, IC3, R1, R2, R3

Commit message: w
Parts:
- added J2: 52806-3010, 52806-3010:528063010, symbol 52806-3010:52806-3010
- IC2: footprint SOT95P275X110-5N -> 74AHC1G86GV,125:SOT95P275X110-5N
- IC3: footprint SOT65P210X110-6N -> MAX9010:SOT65P210X110-6N
Connections:
- net +3.3v is gone; now on net +3.3V: C3.2, C4.2, IC2.5 (VCC), S1.1, S2.1, S3.1, S4.1, S5.1
- net VCC is gone; now on net +3.3V: R2.1
- net DSP_Q0: now also J2.25
- net DSP_Q1: now also J2.24
- net DSP_Q10: now also J2.10
- net DSP_Q11: now also J2.9
- net DSP_Q12: now also J2.7
- net DSP_Q2: now also J2.22
- net DSP_Q3: now also J2.21
- net DSP_Q4: now also J2.19
- net DSP_Q5: now also J2.18
- net DSP_Q6: now also J2.16
- net DSP_Q7: now also J2.15
- net DSP_Q8: now also J2.13
- net DSP_Q9: now also J2.12
- net GND: now also J2.11, J2.14, J2.17, J2.2, J2.20, J2.23, J2.26, J2.29, J2.5, J2.8
- net OUTPUT_ENABLE: now also J2.30
- net Read_CLK: now also J2.1
- net ~{Empty_flag}_Output: now also J2.6
- net ~{Half_full_flag}_Output: now also J2.27
- net ~{Read_enable}: now also J2.3
- net ~{Reset}: now also J2.4
- net ~{Write_enable}: now also J2.28
- no-connect marks 8 -> 19
Other:
- note added: "FIFO fpc cable header"

Commit message: w
Parts:
- removed J2: 52806-3010, 52806-3010:528063010, symbol 52806-3010:52806-3010
- added J3: SFV30R-1STE1HLF, SFV30R1STE1HLF:SFV30R1STE1HLF, symbol SFV30R-1STE1HLF:SFV30R-1STE1HLF
Connections:
- net DSP_Q0: now also J3.25
- net DSP_Q1: now also J3.23
- net DSP_Q10: now also J3.10
- net DSP_Q11: now also J3.8
- net DSP_Q12: now also J3.7
- net DSP_Q2: now also J3.22
- net DSP_Q3: now also J3.20
- net DSP_Q4: now also J3.19
- net DSP_Q5: now also J3.17
- net DSP_Q6: now also J3.16
- net DSP_Q7: now also J3.14
- net DSP_Q8: now also J3.13
- net DSP_Q9: now also J3.11
- net GND: now also J3.1, J3.12, J3.15, J3.18, J3.21, J3.24, J3.27, J3.30, J3.6, J3.9
- net OUTPUT_ENABLE: now also J3.2
- net Read_CLK: now also J3.26
- net ~{Empty_flag}_Output: now also J3.29
- net ~{Half_full_flag}_Output: now also J3.28
- net ~{Read_enable}: now also J3.5
- net ~{Reset}: now also J3.4
- net ~{Write_enable}: now also J3.3
- no-connect marks 19 -> 21
