File: FIFO_FPC_TO_BTB_mini_PCB/FIFO_FPC_TO_BTB_mini_PCB/FIFO_FPC_TO_BTB_mini_PCB.kicad_sch (KiCad schematic)
At the start: 3 parts, among them J1 52806-3010, J2 DF40C_2.0_-60DS-0.4V_51_, J3 52806-3010

Commit message: w
Parts:
- removed J1, J3: 52806-3010, 52806-3010:528063010, symbol 52806-3010:52806-3010
- added J1: SFV30R-1STE1HLF, SFV30R1STE1HLF:SFV30R1STE1HLF, symbol SFV30R-1STE1HLF:SFV30R-1STE1HLF
- J2: footprint DF40C2060DS04V51 -> DF40C2060DS04V51:DF40C2060DS04V51
Connections:
- net GND: now also J2.2, J2.20, J2.30, J2.41, J2.52, J2.9, J1.1, J1.10, J1.13, J1.16, J1.19, J1.22, J1.25, J1.30, J1.4, J1.7
- net hed_~{Half_full_flag}_Output: now reaches J2.10
- net hed_~{Half_full_flag}_Output: now also J1.2
- net Hed_OUTPUT_ENABLE: now reaches J2.12
- net Hed_OUTPUT_ENABLE: now also J1.29
- net hed_~{Write_enable}: now reaches J2.14
- net hed_~{Write_enable}: now also J1.28
- net ~{Hed_Read_enable}: now reaches J2.16
- net ~{Hed_Read_enable}: now also J1.26
- net ~{Hed_Empty_flag}_Output: now reaches J2.18
- net ~{Hed_Empty_flag}_Output: now also J1.3
- net Hed_DSP_Q1: now reaches J2.21
- net Hed_DSP_Q1: now also J1.9
- net Hed_DSP_Q0: now reaches J2.22
- net Hed_DSP_Q0: now also J1.5
- net Hed_DSP_Q3: now reaches J2.23
- net Hed_DSP_Q3: now also J1.12
- net Hed_DSP_Q2: now reaches J2.24
- net Hed_DSP_Q2: now also J1.8
- net Hed_DSP_Q5: now reaches J2.25
- net Hed_DSP_Q5: now also J1.15
- net Hed_DSP_Q4: now reaches J2.26
- net Hed_DSP_Q4: now also J1.11
- net Hed_DSP_Q7: now reaches J2.27
- net Hed_DSP_Q7: now also J1.18
- net Hed_DSP_Q8: now reaches J2.33
- net Hed_DSP_Q8: now also J1.17
- net hed_DSP_Q10: now reaches J2.35
- net hed_DSP_Q10: now also J1.20
- net hed_DSP_Q9: now reaches J2.36
- net hed_DSP_Q9: now also J1.21
- net hed_DSP_Q12: now reaches J2.37
- net hed_DSP_Q12: now also J1.23
- net Hed_DSP_Q11: now reaches J2.38
- net Hed_DSP_Q11: now also J1.24
- net Hed_Read_CLK: now reaches J2.44
- net Hed_Read_CLK: now also J1.27
- net hed_~{Reset}: now reaches J2.6
- net hed_~{Reset}: now also J1.6
- new net hed_DSP_Q6: J1.14
- no-connect marks 0 -> 36
Other:
- note added: "Pin 2 matches with the marker dot"
- note removed: "FIFO fpc cable header needs to be in reverse compared to the inout FPC"

Commit message: w
Connections:
- net Hed_DSP_Q7: now also J1.17; no longer J1.18
- net Hed_DSP_Q8: now also J1.18; no longer J1.17
- net hed_DSP_Q6: now also J2.28
Other:
- moved on the sheet: J1
