File: FIFO_FPC_TO_BTB_mini_PCB/FIFO_FPC_TO_BTB_mini_PCB/FIFO_FPC_TO_BTB_mini_PCB.kicad_pcb (KiCad board)
At the start: 4 copper layers, 2 parts, among them J1 SFV30R-1STE1HLF, J2 DF40C_2.0_-60DS-0.4V_51_

Commit message: w
Parts:
- moved J1 6.67 mm to (151.3, 99.3)
- moved J2 6.67 mm to (120.1, 114.2)
Connections:
- J1 pad 17: /Hed_DSP_Q8 -> /Hed_DSP_Q7
- J1 pad 18: /Hed_DSP_Q7 -> /Hed_DSP_Q8
Routing:
- net GND: track 57.3 -> 62.1 mm
- net /Hed_DSP_Q7: track 41.3 -> 44.3 mm
- net /Hed_DSP_Q1: track 45.6 -> 43.3 mm
- net /Hed_OUTPUT_ENABLE: track 49.0 -> 51.1 mm
- net /~{Hed_Read_enable}: track 46.2 -> 47.5 mm
- net /hed_~{Reset}: track 40.3 -> 41.5 mm
- net /Hed_DSP_Q5: track 44.0 -> 45.1 mm
- net /hed_~{Half_full_flag}_Output: track 35.1 -> 36.2 mm
- net /Hed_DSP_Q3: track 44.8 -> 43.9 mm
- net /~{Hed_Empty_flag}_Output: track 32.4 -> 33.3 mm
- net /hed_~{Write_enable}: track 48.3 -> 49.2 mm
- net /Hed_DSP_Q8: track 44.0 -> 44.8 mm
- net /hed_DSP_Q10: track 43.6 -> 42.9 mm
- net /hed_DSP_Q12: track 43.1 -> 42.6 mm
Other:
- board outline added: 83.5 x 61.5 mm

Commit message: w
Parts:
- moved J1 4.00 mm to (155.3, 99.3)
Routing:
- net GND: track 62.1 -> 70.7 mm, vias 4 -> 5
- net /Hed_DSP_Q0: track 32.8 -> 36.8 mm
- net /Hed_Read_CLK: track 35.2 -> 39.2 mm
- net /Hed_DSP_Q4: track 33.5 -> 37.5 mm
- net /Hed_DSP_Q2: track 33.1 -> 37.1 mm
- net /hed_DSP_Q6: track 33.8 -> 37.8 mm
- net /Hed_DSP_Q11: track 35.1 -> 39.1 mm
- net /hed_DSP_Q9: track 34.6 -> 38.6 mm
- net /hed_DSP_Q10: track 42.9 -> 46.9 mm
- net /Hed_DSP_Q1: track 43.3 -> 47.3 mm
- net /hed_~{Write_enable}: track 49.2 -> 53.1 mm
- net /Hed_DSP_Q3: track 43.9 -> 47.8 mm
- net /Hed_OUTPUT_ENABLE: track 51.1 -> 54.9 mm
- net /~{Hed_Empty_flag}_Output: track 33.3 -> 37.1 mm
- net /hed_DSP_Q12: track 42.6 -> 46.3 mm
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